File: ValveController.kicad_sch (KiCad schematic)
At the start: 52 parts, among them J10 1770966, J11 1770966, J12 1770966, J13 USB4115-03-C, J2 1990986, J3 1990986, J8 1770966, J9 1770966, Q3 MOC3063S-TA1, Q4 MOC3063S-TA1, SW1 TL9320AF400QG, U1 IRM-03-5, U2 TLV75733P, U5 ESP32-C6-WROOM-1-N4

Commit message: fix(sch): rewire D1 active-low, add SSR pull-downs, drop DBG labels
- D1 was reverse-biased (pad1=cathode on driven net) and could never light;
  now 3V3 -> R4 -> anode, cathode -> GPIO15 (also defines JTAG strap high)
- R8/R9 10k pull-downs on SSR_OPEN/SSR_CLOSE define triacs-off at reset
- DBG_TX/DBG_RX labels removed (J15 dropped for good), pins NC-flagged
- ERC hygiene: PWR_FLAGs on mains/5V nets, NC flags on unused GPIOs (94->82)
- Netlist diff verified: only the intended topology changes
Parts:
- added R8, R9: 10k, Resistor_SMD:R_0402_1005Metric, symbol R_dev
- D1: value LED -> LED (active-low)
Connections:
- net 3V3: now also R4.1
- net GND: now also R8.2, R9.2; no longer D1.2
- net LED_A: now also D1.2; no longer D1.1
- net SSR_CLOSE: now also R9.1
- net SSR_OPEN: now also R8.1
- net STAT_LED: now also D1.1; no longer R4.1
- net DBG_RX: no longer names the net of U5.24 (RXD0)
- net DBG_TX: no longer names the net of U5.25 (TXD0)
- no-connect marks 6 -> 17
