File: pcb/ValveController.kicad_sch (KiCad schematic)
At the start: 121 parts, among them J10 1770966, J11 1770966, J12 1770966, J13 USB4145-03-0170-C, J14 1990986, J15 1990999, J2 1990986, J3 1990986, J8 1770966, J9 1770966, Q3 MOC3063S-TA1, Q4 MOC3063S-TA1, Q5 CSD17313Q2, Q6 CPC1035N, Q7 CPC1035N, SW1 TL9320AF400QG, SW3 A6S-1102-H, U1 IRM-03-5, U10 USBLC6-2SC6, U2 TLV75733P, U5 ESP32-C6-WROOM-1-N4, U6 TPS61040, U7 IS31FL3730, U8 HCPL-354-06AE, U9 HCPL-354-06AE

Commit message: feat(pcb): complete 4-layer layout — routing, HV isolation rules, EP thermal vias, board art
Parts:
- added G1: KleistLabs_Logo_8mm_Copper, Kleist2:KleistLabs_Logo_8mm_Copper, symbol Kleist2:KleistLabs_Logo_8mm_Copper
- added G2: QR_HydroMix_SilkOnDark, Kleist2:QR_HydroMix_250um_SilkOnDark, symbol Kleist2:QR_HydroMix_SilkOnDark
- C14, C16, C17, C2, C20, C7, C8: DigiKey https://www.digikey.com/en/products/detail/murata-electroni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 -> https://www.digikey.com/en/products/detail/samsung-electro-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; MPN GRM155R71C104KA88D -> CL05B104KO5NNNC
- C4, C5, C6: DigiKey https://www.digikey.com/en/products/detail/samsung-electro-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 -> https://www.digikey.com/en/products/detail/kemet/C0805C106K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; MPN CL21A106KOFNNNE -> C0805C106K3PACTU
- H1, H3, H4: footprint MountingHole:MountingHole_3.2mm_M3_DIN965_Pad -> MountingHole:MountingHole_3.2mm_M3_ISO7380
- H2: footprint MountingHole:MountingHole_3.2mm_M3_DIN965_Pad -> MountingHole:MountingHole_3.2mm_M3_ISO7380; symbol Mechanical:MountingHole -> Mechanical:MountingHole_Pad
Other:
- moved on the sheet: R40
